Commit message: update jazzy code

File: mobo_bot_description/urdf/gazebo_properties.xacro (robot description, xacro)
@@ -192,5 +192,5 @@
     <sensor name="camera_optical" type="camera">
     <!-- <sensor name="camera_optical" type="depth"> -->
-      <gz_frame_id>camera</gz_frame_id>
+      <gz_frame_id>camera_optical</gz_frame_id>
       <camera>
         <horizontal_fov>1.047</horizontal_fov>
@@ -213,6 +213,6 @@
   <gazebo>
     <plugin
-      filename="ignition-gazebo-diff-drive-system"
-      name="ignition::gazebo::systems::DiffDrive">
+      filename="gz-sim-diff-drive-system"
+      name="gz::sim::systems::DiffDrive">
       <left_joint>left_wheel_joint</left_joint>
       <right_joint>right_wheel_joint</right_joint>
@@ -234,7 +234,7 @@
   <gazebo>
     <plugin
-      filename="ignition-gazebo-odometry-publisher-system"
-      name="ignition::gazebo::systems::OdometryPublisher">
-      <odom_publish_frequency>30</odom_publish_frequency>
+      filename="gz-sim-odometry-publisher-system"
+      name="gz::sim::systems::OdometryPublisher">
+      <odom_publish_frequency>70</odom_publish_frequency>
       <robot_base_frame>base_link</robot_base_frame>
       <odom_frame>odom</odom_frame>
@@ -243,6 +243,6 @@
   <gazebo>
     <plugin
-      filename="ignition-gazebo-joint-state-publisher-system"
-      name="ignition::gazebo::systems::JointStatePublisher">
+      filename="gz-sim-joint-state-publisher-system"
+      name="gz::sim::systems::JointStatePublisher">
       <joint_name>left_wheel_joint</joint_name>
       <joint_name>right_wheel_joint</joint_name>

File: mobo_bot_description/urdf/robot_urdf.xacro (robot description, xacro)
@@ -53,15 +53,15 @@
     <xacro:include filename="$(find mobo_bot_description)/urdf/urdf_models/lidar.xacro"/>
     <xacro:include filename="$(find mobo_bot_description)/urdf/urdf_models/cam.xacro"/>
-    <xacro:property name="chassis_length" value="0.21"/>
-    <xacro:property name="chassis_width" value="0.21"/>
-    <xacro:property name="chassis_height" value="0.06"/>
+    <xacro:property name="chassis_length" value="0.20"/>
+    <xacro:property name="chassis_width" value="0.20"/>
+    <xacro:property name="chassis_height" value="0.05"/>
     <xacro:property name="slab_height" value="0.005"/>
     <xacro:property name="chassis_mass" value="2.0"/>
     <xacro:property name="chassis_color" value="orange"/>
-    <xacro:property name="wheel_seperation" value="0.24"/>
+    <xacro:property name="wheel_seperation" value="0.225"/>
     <xacro:property name="wheel_radius" value="0.034"/>
-    <xacro:property name="wheel_width" value="0.026"/>
+    <xacro:property name="wheel_width" value="0.014"/>
     <xacro:property name="wheel_mass" value="0.08"/>
-    <xacro:property name="wheel_height_offset" value="0.024"/>
+    <xacro:property name="wheel_height_offset" value="0.015"/>
     <xacro:property name="castor_wheel_diameter" value="${wheel_radius+wheel_height_offset}"/>
     <xacro:property name="castor_wheel_mass" value="0.08"/>
@@ -76,8 +76,8 @@
         <xacro:insert_box_with_fillet x="-0.040" y="0" z="0"
             size_x="${chassis_length}" size_y="${chassis_width}" size_z="${slab_height}"
-            fillet_radius="0.04"/>
+            fillet_radius="0.02"/>
         <xacro:insert_box_with_fillet x="-0.040" y="0" z="${chassis_height}"
             size_x="${chassis_length}" size_y="${chassis_width}" size_z="${slab_height}"
-            fillet_radius="0.04"/>
+            fillet_radius="0.02"/>
         <visual>
             <origin xyz="0.04 0.08 ${chassis_height/2}" rpy="0 0 0"/>
@@ -195,5 +195,5 @@
     </xacro:if>
     <xacro:unless value="$(arg run_gz_sim)">
-        <xacro:include filename="$(find mobo_bot_description)/urdf/epmc_ros2_control.xacro" />
+        <xacro:include filename="$(find mobo_bot_description)/urdf/ros2_control.xacro" />
     </xacro:unless>
 </robot>
