Commit message: added option for using for wheel diff drive mobo_bot

File: mobo_bot_description/urdf/robot_urdf.xacro (robot description, xacro)
@@ -2,4 +2,5 @@
 <robot name="mobo_bot" xmlns:xacro="http://www.ros.org/wiki/xacro">
     <xacro:arg name="run_gz_sim" default="false"/>
+    <xacro:arg name="use_4_wheels" default="false"/>
     <material name="orange">
         <color rgba="1 0.55 0 1"/>
@@ -47,153 +48,21 @@
         </inertial>
     </xacro:macro>
-    <xacro:include filename="$(find mobo_bot_description)/urdf/urdf_models/box_with_fillet_macro.xacro"/>
-    <xacro:include filename="$(find mobo_bot_description)/urdf/urdf_models/drive_wheel_macro.xacro"/>
-    <xacro:include filename="$(find mobo_bot_description)/urdf/urdf_models/drive_wheel_rim_macro.xacro"/>
-    <xacro:include filename="$(find mobo_bot_description)/urdf/urdf_models/sonar.xacro"/>
-    <xacro:include filename="$(find mobo_bot_description)/urdf/urdf_models/lidar.xacro"/>
-    <xacro:include filename="$(find mobo_bot_description)/urdf/urdf_models/cam.xacro"/>
-    <xacro:property name="chassis_length" value="0.20"/>
-    <xacro:property name="chassis_width" value="0.20"/>
-    <xacro:property name="chassis_height" value="0.05"/>
-    <xacro:property name="slab_height" value="0.005"/>
-    <xacro:property name="chassis_mass" value="2.0"/>
-    <xacro:property name="chassis_color" value="orange"/>
-    <xacro:property name="wheel_seperation" value="0.225"/>
-    <xacro:property name="wheel_radius" value="0.034"/>
-    <xacro:property name="wheel_width" value="0.014"/>
-    <xacro:property name="wheel_mass" value="0.08"/>
-    <xacro:property name="wheel_height_offset" value="0.015"/>
-    <xacro:property name="castor_wheel_diameter" value="${wheel_radius+wheel_height_offset}"/>
-    <xacro:property name="castor_wheel_mass" value="0.08"/>
-    <link name="base_link">
-    </link>
-    <joint name="chassis_joint" type="fixed">
-        <parent link="base_link"/>
-        <child link="chassis"/>
-        <origin xyz="0 0 ${wheel_radius+wheel_height_offset}"/>
-    </joint>
-    <link name="chassis">
-        <xacro:insert_box_with_fillet x="-0.040" y="0" z="0"
-            size_x="${chassis_length}" size_y="${chassis_width}" size_z="${slab_height}"
-            fillet_radius="0.02"/>
-        <xacro:insert_box_with_fillet x="-0.040" y="0" z="${chassis_height}"
-            size_x="${chassis_length}" size_y="${chassis_width}" size_z="${slab_height}"
-            fillet_radius="0.02"/>
-        <visual>
-            <origin xyz="0.04 0.08 ${chassis_height/2}" rpy="0 0 0"/>
-            <geometry>
-                <cylinder radius="0.005" length="${chassis_height}"/>
-            </geometry>
-            <material name="orange"/>
-        </visual>
-        <visual>
-            <origin xyz="0.04 -0.08 ${chassis_height/2}" rpy="0 0 0"/>
-            <geometry>
-                <cylinder radius="0.005" length="${chassis_height}"/>
-            </geometry>
-            <material name="orange"/>
-        </visual>
-        <visual>
-            <origin xyz="-0.11 0.08 ${chassis_height/2}" rpy="0 0 0"/>
-            <geometry>
-                <cylinder radius="0.005" length="${chassis_height}"/>
-            </geometry>
-            <material name="orange"/>
-        </visual>
-        <visual>
-            <origin xyz="-0.11 -0.08 ${chassis_height/2}" rpy="0 0 0"/>
-            <geometry>
-                <cylinder radius="0.005" length="${chassis_height}"/>
-            </geometry>
-            <material name="orange"/>
-        </visual>
-        <collision>
-           <origin xyz="-0.02 0 ${chassis_height/2}" rpy="0 0 0"/>
-            <geometry>
-                <box size="${chassis_length} ${chassis_width} ${chassis_height}"/>
-            </geometry>
-        </collision>
-        <xacro:inertial_box mass="${chassis_mass}" x="${chassis_length}" y="${chassis_width}" z="${chassis_height}">
-            <origin xyz="-0.06 0 ${chassis_height/2}" rpy="0 0 0"/>
-        </xacro:inertial_box>
-    </link>
-    <xacro:insert_drive_wheel
-        base_name="left_wheel"
-        parent_name="base_link"
-        x="0" y="${wheel_seperation/2}" z="${wheel_radius}"
-        mass="${wheel_mass}"
-        radius="${wheel_radius}"
-        thickness="${wheel_width}"/>
-    <xacro:insert_drive_wheel_rim
-        base_name="left_rim"
-        parent_name="left_wheel"
-        radius="${wheel_radius}"
-        thickness="${wheel_width}"
-        spoke_width="0.005"/>
-    <xacro:insert_drive_wheel
-        base_name="right_wheel"
-        parent_name="base_link"
-        x="0" y="${-wheel_seperation/2}" z="${wheel_radius}"
-        mass="${wheel_mass}"
-        radius="${wheel_radius}"
-        thickness="${wheel_width}"/>
-    <xacro:insert_drive_wheel_rim
-        base_name="right_rim"
-        parent_name="right_wheel"
-        radius="${wheel_radius}"
-        thickness="${wheel_width}"
-        spoke_width="0.005"/>
-    <joint name="castor_wheel_joint" type="fixed">
-        <parent link="base_link"/>
-        <child link="castor_wheel"/>
-        <origin xyz="-0.1 0 ${castor_wheel_diameter/2}"/>
-    </joint>
-    <link name="castor_wheel">
-        <visual>
-            <origin xyz="0 0 0" rpy="0 0 0"/>
-            <geometry>
-                <sphere radius="${castor_wheel_diameter/2}" />
-            </geometry>
-            <material name="grey">
-                <color rgba="0.25 0.25 0.25 1"/>
-            </material>
-        </visual>
-        <collision>
-           <origin xyz="0 0 0" rpy="0 0 0"/>
-            <geometry>
-                <sphere radius="${castor_wheel_diameter/2}" />
-            </geometry>
-        </collision>
-        <xacro:inertial_sphere mass="${castor_wheel_mass}" radius="${castor_wheel_diameter/2}">
-            <origin xyz="0 0 0" rpy="0 0 0"/>
-        </xacro:inertial_sphere>
-    </link>
-    <xacro:property name="lidar_z_offset" value="0.04"/>
-    <xacro:insert_lidar
-        base_name="lidar"
-        parent_name="chassis"
-        x="0.01" y="0" z="${chassis_height+lidar_z_offset}"
-        mass="0.1"/>
-    <joint name="imu_joint" type="fixed">
-        <parent link="chassis"/>
-        <child link="imu"/>
-        <origin xyz="0 0 ${chassis_height}"/>
-    </joint>
-    <link name="imu"></link>
-    <xacro:insert_sonar
-        base_name="sonar"
-        parent_name="chassis"
-        x="0.065" y="0" z="${chassis_height/6}"
-        mass="0.005"/>
-    <xacro:insert_camera
-        base_name="camera"
-        parent_name="chassis"
-        x="0.075" y="0" z="${chassis_height+0.015}"
-        mass="0.005" tilt_angle="0.00"/>
-    <xacro:if value="$(arg run_gz_sim)">
-        <xacro:include filename="$(find mobo_bot_description)/urdf/gazebo_properties.xacro" />
+    <xacro:if value="$(arg use_4_wheels)">
+        <xacro:include filename="$(find mobo_bot_description)/urdf/four_wheel_base/robot.xacro" />
+        <xacro:if value="$(arg run_gz_sim)">
+            <xacro:include filename="$(find mobo_bot_description)/urdf/four_wheel_base/gazebo_properties.xacro" />
+        </xacro:if>
+        <xacro:unless value="$(arg run_gz_sim)">
+            <xacro:include filename="$(find mobo_bot_description)/urdf/four_wheel_base/ros2_control.xacro" />
+        </xacro:unless>
     </xacro:if>
-    <xacro:unless value="$(arg run_gz_sim)">
-        <xacro:include filename="$(find mobo_bot_description)/urdf/ros2_control.xacro" />
+    <xacro:unless value="$(arg use_4_wheels)">
+        <xacro:include filename="$(find mobo_bot_description)/urdf/two_wheel_base/robot.xacro" />
+        <xacro:if value="$(arg run_gz_sim)">
+            <xacro:include filename="$(find mobo_bot_description)/urdf/two_wheel_base/gazebo_properties.xacro" />
+        </xacro:if>
+        <xacro:unless value="$(arg run_gz_sim)">
+            <xacro:include filename="$(find mobo_bot_description)/urdf/two_wheel_base/ros2_control.xacro" />
+        </xacro:unless>
     </xacro:unless>
 </robot>

File: mobo_bot_description/urdf/two_wheel_base/gazebo_properties.xacro (robot description, xacro)
@@ -197,5 +197,5 @@
         <image>
           <width>640</width>
-          <height>360</height>
+          <height>480</height>
         </image>
         <clip>
@@ -217,5 +217,5 @@
       <left_joint>left_wheel_joint</left_joint>
       <right_joint>right_wheel_joint</right_joint>
-      <wheel_separation>0.25</wheel_separation>
+      <wheel_separation>0.236</wheel_separation>
       <wheel_radius>0.034</wheel_radius>
       <!--
@@ -236,5 +236,5 @@
       filename="gz-sim-odometry-publisher-system"
       name="gz::sim::systems::OdometryPublisher">
-      <odom_publish_frequency>70</odom_publish_frequency>
+      <odom_publish_frequency>60</odom_publish_frequency>
       <robot_base_frame>base_link</robot_base_frame>
       <odom_frame>odom</odom_frame>

File: mobo_bot_description/urdf/two_wheel_base/ros2_control.xacro (robot description, xacro)
@@ -4,14 +4,13 @@
       <hardware>
         <plugin>epmc_v2_hardware_interface/EPMC_V2_HardwareInterface</plugin>
-        <!-- <param name="port">/dev/ttyUSB0</param> -->
         <param name="port">/dev/epmc</param>
         <param name="motor0_wheel_name">left_wheel_joint</param>
         <param name="motor1_wheel_name">right_wheel_joint</param>
-        <param name="cmd_vel_timeout_ms">2000</param>
+        <param name="cmd_vel_timeout_ms">5000</param>
       </hardware>
       <joint name="left_wheel_joint">
         <command_interface name="velocity">
-            <param name="min">-10.0</param>
-            <param name="max">10.0</param>
+            <param name="min">-16.0</param>
+            <param name="max">16.0</param>
         </command_interface>
         <state_interface name="position"/>
@@ -20,6 +19,6 @@
       <joint name="right_wheel_joint">
         <command_interface name="velocity">
-            <param name="min">-10.0</param>
-            <param name="max">10.0</param>
+            <param name="min">-16.0</param>
+            <param name="max">16.0</param>
         </command_interface>
         <state_interface name="position"/>

Commit message: update how base are selected

File: mobo_bot_description/urdf/robot_urdf.xacro (robot description, xacro)
@@ -2,5 +2,6 @@
 <robot name="mobo_bot" xmlns:xacro="http://www.ros.org/wiki/xacro">
     <xacro:arg name="run_gz_sim" default="false"/>
-    <xacro:arg name="use_4_wheels" default="false"/>
+    <xacro:arg name="wheel_type" default="2wheel"/>
+    <xacro:property name="wheel_type_name" value="$(arg wheel_type)"/>
     <material name="orange">
         <color rgba="1 0.55 0 1"/>
@@ -48,5 +49,6 @@
         </inertial>
     </xacro:macro>
-    <xacro:if value="$(arg use_4_wheels)">
+    <!-- Conditional inclusion -->
+    <xacro:if value="${wheel_type_name == '4wheel'}">
         <xacro:include filename="$(find mobo_bot_description)/urdf/four_wheel_base/robot.xacro" />
         <xacro:if value="$(arg run_gz_sim)">
@@ -57,5 +59,5 @@
         </xacro:unless>
     </xacro:if>
-    <xacro:unless value="$(arg use_4_wheels)">
+    <xacro:if value="${wheel_type_name == '2wheel'}">
         <xacro:include filename="$(find mobo_bot_description)/urdf/two_wheel_base/robot.xacro" />
         <xacro:if value="$(arg run_gz_sim)">
@@ -65,4 +67,4 @@
             <xacro:include filename="$(find mobo_bot_description)/urdf/two_wheel_base/ros2_control.xacro" />
         </xacro:unless>
-    </xacro:unless>
+    </xacro:if>
 </robot>
