Commit message: update robot design

File: mobo_bot_description/urdf/four_wheel_base/gazebo_properties.xacro (robot description, xacro)
@@ -182,6 +182,6 @@
           <horizontal>
             <samples>360</samples>
-            <min_angle>${-pi}</min_angle>
-            <max_angle>${pi}</max_angle>
+            <min_angle>${-0.833*pi}</min_angle>
+            <max_angle>${0.833*pi}</max_angle>
             <resolution>1</resolution>
           </horizontal>

File: mobo_bot_description/urdf/four_wheel_base/robot.xacro (robot description, xacro)
@@ -7,5 +7,5 @@
     <xacro:include filename="$(find mobo_bot_description)/urdf/urdf_models/lidar.xacro"/>
     <xacro:include filename="$(find mobo_bot_description)/urdf/urdf_models/cam.xacro"/>
-    <xacro:property name="chassis_length" value="0.20"/>
+    <xacro:property name="chassis_length" value="0.24"/>
     <xacro:property name="chassis_width" value="0.20"/>
     <xacro:property name="chassis_height" value="0.05"/>
@@ -18,5 +18,5 @@
     <xacro:property name="wheel_mass" value="0.08"/>
     <xacro:property name="wheel_height_offset" value="0.025"/>
-    <xacro:property name="wheel_base_dist" value="0.12"/>
+    <xacro:property name="wheel_base_dist" value="0.14"/>
     <link name="base_link">
     </link>
@@ -29,10 +29,10 @@
         <xacro:insert_box_with_fillet x="0" y="0" z="0"
             size_x="${chassis_length}" size_y="${chassis_width}" size_z="${slab_height}"
-            fillet_radius="0.02"/>
+            fillet_radius="0.025"/>
         <xacro:insert_box_with_fillet x="0" y="0" z="${chassis_height}"
             size_x="${chassis_length}" size_y="${chassis_width}" size_z="${slab_height}"
             fillet_radius="0.02"/>
         <visual>
-            <origin xyz="0.08 0.08 ${chassis_height/2}" rpy="0 0 0"/>
+            <origin xyz="0.1 0.08 ${chassis_height/2}" rpy="0 0 0"/>
             <geometry>
                 <cylinder radius="0.005" length="${chassis_height}"/>
@@ -41,5 +41,5 @@
         </visual>
         <visual>
-            <origin xyz="0.08 -0.08 ${chassis_height/2}" rpy="0 0 0"/>
+            <origin xyz="0.1 -0.08 ${chassis_height/2}" rpy="0 0 0"/>
             <geometry>
                 <cylinder radius="0.005" length="${chassis_height}"/>
@@ -48,5 +48,5 @@
         </visual>
         <visual>
-            <origin xyz="-0.08 0.08 ${chassis_height/2}" rpy="0 0 0"/>
+            <origin xyz="-0.1 0.08 ${chassis_height/2}" rpy="0 0 0"/>
             <geometry>
                 <cylinder radius="0.005" length="${chassis_height}"/>
@@ -55,5 +55,5 @@
         </visual>
         <visual>
-            <origin xyz="-0.08 -0.08 ${chassis_height/2}" rpy="0 0 0"/>
+            <origin xyz="-0.1 -0.08 ${chassis_height/2}" rpy="0 0 0"/>
             <geometry>
                 <cylinder radius="0.005" length="${chassis_height}"/>
@@ -127,5 +127,5 @@
         base_name="lidar"
         parent_name="chassis"
-        x="0.04" y="0" z="${chassis_height+lidar_z_offset}"
+        x="0.05" y="0" z="${chassis_height+lidar_z_offset}"
         mass="0.1"/>
     <joint name="imu_joint" type="fixed">
@@ -138,10 +138,10 @@
         base_name="sonar"
         parent_name="chassis"
-        x="0.1" y="0" z="${chassis_height/6}"
+        x="0.12" y="0" z="${chassis_height/6}"
         mass="0.005"/>
     <xacro:insert_camera
         base_name="camera"
         parent_name="chassis"
-        x="0.12" y="0" z="${chassis_height+0.015}"
+        x="0.14" y="0" z="${chassis_height+0.015}"
         mass="0.005" tilt_angle="0.00"/>
 </robot>

File: mobo_bot_description/urdf/two_wheel_base/gazebo_properties.xacro (robot description, xacro)
@@ -165,6 +165,6 @@
           <horizontal>
             <samples>360</samples>
-            <min_angle>${-pi}</min_angle>
-            <max_angle>${pi}</max_angle>
+            <min_angle>${-0.833*pi}</min_angle>
+            <max_angle>${0.833*pi}</max_angle>
             <resolution>1</resolution>
           </horizontal>

File: mobo_bot_description/urdf/two_wheel_base/robot.xacro (robot description, xacro)
@@ -7,5 +7,5 @@
     <xacro:include filename="$(find mobo_bot_description)/urdf/urdf_models/lidar.xacro"/>
     <xacro:include filename="$(find mobo_bot_description)/urdf/urdf_models/cam.xacro"/>
-    <xacro:property name="chassis_length" value="0.20"/>
+    <xacro:property name="chassis_length" value="0.24"/>
     <xacro:property name="chassis_width" value="0.20"/>
     <xacro:property name="chassis_height" value="0.05"/>
@@ -35,5 +35,5 @@
             fillet_radius="0.02"/>
         <visual>
-            <origin xyz="0.04 0.08 ${chassis_height/2}" rpy="0 0 0"/>
+            <origin xyz="0.06 0.08 ${chassis_height/2}" rpy="0 0 0"/>
             <geometry>
                 <cylinder radius="0.005" length="${chassis_height}"/>
@@ -42,5 +42,5 @@
         </visual>
         <visual>
-            <origin xyz="0.04 -0.08 ${chassis_height/2}" rpy="0 0 0"/>
+            <origin xyz="0.06 -0.08 ${chassis_height/2}" rpy="0 0 0"/>
             <geometry>
                 <cylinder radius="0.005" length="${chassis_height}"/>
@@ -49,5 +49,5 @@
         </visual>
         <visual>
-            <origin xyz="-0.11 0.08 ${chassis_height/2}" rpy="0 0 0"/>
+            <origin xyz="-0.14 0.08 ${chassis_height/2}" rpy="0 0 0"/>
             <geometry>
                 <cylinder radius="0.005" length="${chassis_height}"/>
@@ -56,5 +56,5 @@
         </visual>
         <visual>
-            <origin xyz="-0.11 -0.08 ${chassis_height/2}" rpy="0 0 0"/>
+            <origin xyz="-0.14 -0.08 ${chassis_height/2}" rpy="0 0 0"/>
             <geometry>
                 <cylinder radius="0.005" length="${chassis_height}"/>
@@ -63,5 +63,5 @@
         </visual>
         <collision>
-           <origin xyz="-0.02 0 ${chassis_height/2}" rpy="0 0 0"/>
+           <origin xyz="-0.04 0 ${chassis_height/2}" rpy="0 0 0"/>
             <geometry>
                 <box size="${chassis_length} ${chassis_width} ${chassis_height}"/>
@@ -69,5 +69,5 @@
         </collision>
         <xacro:inertial_box mass="${chassis_mass}" x="${chassis_length}" y="${chassis_width}" z="${chassis_height}">
-            <origin xyz="-0.06 0 ${chassis_height/2}" rpy="0 0 0"/>
+            <origin xyz="-0.08 0 ${chassis_height/2}" rpy="0 0 0"/>
         </xacro:inertial_box>
     </link>
@@ -101,5 +101,5 @@
         <parent link="base_link"/>
         <child link="castor_wheel"/>
-        <origin xyz="-0.1 0 ${castor_wheel_diameter/2}"/>
+        <origin xyz="-0.11 0 ${castor_wheel_diameter/2}"/>
     </joint>
     <link name="castor_wheel">
@@ -138,10 +138,10 @@
         base_name="sonar"
         parent_name="chassis"
-        x="0.065" y="0" z="${chassis_height/6}"
+        x="0.08" y="0" z="${chassis_height/6}"
         mass="0.005"/>
     <xacro:insert_camera
         base_name="camera"
         parent_name="chassis"
-        x="0.075" y="0" z="${chassis_height+0.015}"
+        x="0.09" y="0" z="${chassis_height+0.015}"
         mass="0.005" tilt_angle="0.00"/>
 </robot>
