Commit message: update robot design

File: mobo_bot_description/urdf/four_wheel_base/robot.xacro (robot description, xacro)
@@ -7,5 +7,5 @@
     <xacro:include filename="$(find mobo_bot_description)/urdf/urdf_models/lidar.xacro"/>
     <xacro:include filename="$(find mobo_bot_description)/urdf/urdf_models/cam.xacro"/>
-    <xacro:property name="chassis_length" value="0.24"/>
+    <xacro:property name="chassis_length" value="0.22"/>
     <xacro:property name="chassis_width" value="0.20"/>
     <xacro:property name="chassis_height" value="0.05"/>
@@ -18,5 +18,5 @@
     <xacro:property name="wheel_mass" value="0.08"/>
     <xacro:property name="wheel_height_offset" value="0.025"/>
-    <xacro:property name="wheel_base_dist" value="0.14"/>
+    <xacro:property name="wheel_base_dist" value="0.12"/>
     <link name="base_link">
     </link>
@@ -34,28 +34,28 @@
             fillet_radius="0.02"/>
         <visual>
-            <origin xyz="0.1 0.08 ${chassis_height/2}" rpy="0 0 0"/>
+            <origin xyz="0.09 0.08 ${chassis_height/2}" rpy="0 0 0"/>
             <geometry>
-                <cylinder radius="0.005" length="${chassis_height}"/>
+                <cylinder radius="0.004" length="${chassis_height}"/>
             </geometry>
             <material name="orange"/>
         </visual>
         <visual>
-            <origin xyz="0.1 -0.08 ${chassis_height/2}" rpy="0 0 0"/>
+            <origin xyz="0.09 -0.08 ${chassis_height/2}" rpy="0 0 0"/>
             <geometry>
-                <cylinder radius="0.005" length="${chassis_height}"/>
+                <cylinder radius="0.004" length="${chassis_height}"/>
             </geometry>
             <material name="orange"/>
         </visual>
         <visual>
-            <origin xyz="-0.1 0.08 ${chassis_height/2}" rpy="0 0 0"/>
+            <origin xyz="-0.09 0.08 ${chassis_height/2}" rpy="0 0 0"/>
             <geometry>
-                <cylinder radius="0.005" length="${chassis_height}"/>
+                <cylinder radius="0.004" length="${chassis_height}"/>
             </geometry>
             <material name="orange"/>
         </visual>
         <visual>
-            <origin xyz="-0.1 -0.08 ${chassis_height/2}" rpy="0 0 0"/>
+            <origin xyz="-0.09 -0.08 ${chassis_height/2}" rpy="0 0 0"/>
             <geometry>
-                <cylinder radius="0.005" length="${chassis_height}"/>
+                <cylinder radius="0.004" length="${chassis_height}"/>
             </geometry>
             <material name="orange"/>
@@ -138,10 +138,10 @@
         base_name="sonar"
         parent_name="chassis"
-        x="0.12" y="0" z="${chassis_height/6}"
+        x="0.11" y="0" z="${chassis_height/6}"
         mass="0.005"/>
     <xacro:insert_camera
         base_name="camera"
         parent_name="chassis"
-        x="0.14" y="0" z="${chassis_height+0.015}"
+        x="0.13" y="0" z="${chassis_height+0.015}"
         mass="0.005" tilt_angle="0.00"/>
 </robot>

File: mobo_bot_description/urdf/two_wheel_base/robot.xacro (robot description, xacro)
@@ -7,5 +7,5 @@
     <xacro:include filename="$(find mobo_bot_description)/urdf/urdf_models/lidar.xacro"/>
     <xacro:include filename="$(find mobo_bot_description)/urdf/urdf_models/cam.xacro"/>
-    <xacro:property name="chassis_length" value="0.24"/>
+    <xacro:property name="chassis_length" value="0.22"/>
     <xacro:property name="chassis_width" value="0.20"/>
     <xacro:property name="chassis_height" value="0.05"/>
@@ -35,28 +35,28 @@
             fillet_radius="0.02"/>
         <visual>
-            <origin xyz="0.06 0.08 ${chassis_height/2}" rpy="0 0 0"/>
+            <origin xyz="0.05 0.08 ${chassis_height/2}" rpy="0 0 0"/>
             <geometry>
-                <cylinder radius="0.005" length="${chassis_height}"/>
+                <cylinder radius="0.004" length="${chassis_height}"/>
             </geometry>
             <material name="orange"/>
         </visual>
         <visual>
-            <origin xyz="0.06 -0.08 ${chassis_height/2}" rpy="0 0 0"/>
+            <origin xyz="0.05 -0.08 ${chassis_height/2}" rpy="0 0 0"/>
             <geometry>
-                <cylinder radius="0.005" length="${chassis_height}"/>
+                <cylinder radius="0.004" length="${chassis_height}"/>
             </geometry>
             <material name="orange"/>
         </visual>
         <visual>
-            <origin xyz="-0.14 0.08 ${chassis_height/2}" rpy="0 0 0"/>
+            <origin xyz="-0.13 0.08 ${chassis_height/2}" rpy="0 0 0"/>
             <geometry>
-                <cylinder radius="0.005" length="${chassis_height}"/>
+                <cylinder radius="0.004" length="${chassis_height}"/>
             </geometry>
             <material name="orange"/>
         </visual>
         <visual>
-            <origin xyz="-0.14 -0.08 ${chassis_height/2}" rpy="0 0 0"/>
+            <origin xyz="-0.13 -0.08 ${chassis_height/2}" rpy="0 0 0"/>
             <geometry>
-                <cylinder radius="0.005" length="${chassis_height}"/>
+                <cylinder radius="0.004" length="${chassis_height}"/>
             </geometry>
             <material name="orange"/>
@@ -69,5 +69,5 @@
         </collision>
         <xacro:inertial_box mass="${chassis_mass}" x="${chassis_length}" y="${chassis_width}" z="${chassis_height}">
-            <origin xyz="-0.08 0 ${chassis_height/2}" rpy="0 0 0"/>
+            <origin xyz="-0.07 0 ${chassis_height/2}" rpy="0 0 0"/>
         </xacro:inertial_box>
     </link>
@@ -101,5 +101,5 @@
         <parent link="base_link"/>
         <child link="castor_wheel"/>
-        <origin xyz="-0.11 0 ${castor_wheel_diameter/2}"/>
+        <origin xyz="-0.10 0 ${castor_wheel_diameter/2}"/>
     </joint>
     <link name="castor_wheel">
@@ -138,5 +138,5 @@
         base_name="sonar"
         parent_name="chassis"
-        x="0.08" y="0" z="${chassis_height/6}"
+        x="0.07" y="0" z="${chassis_height/6}"
         mass="0.005"/>
     <xacro:insert_camera
