Commit message: update main branch codes

File: mobo_bot_description/urdf/four_wheel_base/ros2_control.xacro (robot description, xacro)
@@ -1,42 +1,31 @@
 <?xml version="1.0"?>
 <robot xmlns:xacro="http://www.ros.org/wiki/xacro">
-    <ros2_control name="epmc_v2_hardware_interface" type="system">
+    <ros2_control name="epmc_hardware_interface" type="system">
       <hardware>
+        <plugin>epmc_hardware_interface/EPMC_HardwareInterface</plugin>
+        <param name="port">/dev/epmc</param>
+        <param name="motorA_wheel_name">left_wheel_joint</param>
+        <param name="motorB_wheel_name">right_wheel_joint</param>
+        <param name="cmd_vel_timeout_ms">2000</param>
+      </hardware>
+      <!-- <hardware>
         <plugin>epmc_v2_hardware_interface/EPMC_V2_HardwareInterface</plugin>
         <param name="port">/dev/epmc</param>
-        <param name="motor0_wheel_name">front_left_wheel_joint</param>
-        <param name="motor1_wheel_name">front_right_wheel_joint</param>
-        <param name="motor2_wheel_name">rear_left_wheel_joint</param>
-        <param name="motor3_wheel_name">rear_right_wheel_joint</param>
-        <param name="cmd_vel_timeout_ms">5000</param>
-      </hardware>
-      <joint name="front_left_wheel_joint">
+        <param name="motor0_wheel_name">left_wheel_joint</param>
+        <param name="motor1_wheel_name">right_wheel_joint</param>
+        <param name="cmd_vel_timeout_ms">2000</param>
+      </hardware> -->
+      <joint name="left_wheel_joint">
         <command_interface name="velocity">
-            <param name="min">-16.0</param>
-            <param name="max">16.0</param>
+            <param name="min">-15.0</param>
+            <param name="max">15.0</param>
         </command_interface>
         <state_interface name="position"/>
         <state_interface name="velocity"/>
       </joint>
-      <joint name="front_right_wheel_joint">
+      <joint name="right_wheel_joint">
         <command_interface name="velocity">
-            <param name="min">-16.0</param>
-            <param name="max">16.0</param>
-        </command_interface>
-        <state_interface name="position"/>
-        <state_interface name="velocity"/>
-      </joint>
-      <joint name="rear_left_wheel_joint">
-        <command_interface name="velocity">
-            <param name="min">-16.0</param>
-            <param name="max">16.0</param>
-        </command_interface>
-        <state_interface name="position"/>
-        <state_interface name="velocity"/>
-      </joint>
-      <joint name="rear_right_wheel_joint">
-        <command_interface name="velocity">
-            <param name="min">-16.0</param>
-            <param name="max">16.0</param>
+            <param name="min">-15.0</param>
+            <param name="max">15.0</param>
         </command_interface>
         <state_interface name="position"/>

File: mobo_bot_description/urdf/two_wheel_base/ros2_control.xacro (robot description, xacro)
@@ -5,20 +5,38 @@
         <plugin>epmc_v2_hardware_interface/EPMC_V2_HardwareInterface</plugin>
         <param name="port">/dev/epmc</param>
-        <param name="motor0_wheel_name">left_wheel_joint</param>
-        <param name="motor1_wheel_name">right_wheel_joint</param>
-        <param name="cmd_vel_timeout_ms">5000</param>
+        <param name="motor0_wheel_name">front_left_wheel_joint</param>
+        <param name="motor1_wheel_name">front_right_wheel_joint</param>
+        <param name="motor2_wheel_name">rear_left_wheel_joint</param>
+        <param name="motor3_wheel_name">rear_right_wheel_joint</param>
+        <param name="cmd_vel_timeout_ms">2000</param>
       </hardware>
-      <joint name="left_wheel_joint">
+      <joint name="front_left_wheel_joint">
         <command_interface name="velocity">
-            <param name="min">-16.0</param>
-            <param name="max">16.0</param>
+            <param name="min">-15.0</param>
+            <param name="max">15.0</param>
         </command_interface>
         <state_interface name="position"/>
         <state_interface name="velocity"/>
       </joint>
-      <joint name="right_wheel_joint">
+      <joint name="front_right_wheel_joint">
         <command_interface name="velocity">
-            <param name="min">-16.0</param>
-            <param name="max">16.0</param>
+            <param name="min">-15.0</param>
+            <param name="max">15.0</param>
+        </command_interface>
+        <state_interface name="position"/>
+        <state_interface name="velocity"/>
+      </joint>
+      <joint name="rear_left_wheel_joint">
+        <command_interface name="velocity">
+            <param name="min">-15.0</param>
+            <param name="max">15.0</param>
+        </command_interface>
+        <state_interface name="position"/>
+        <state_interface name="velocity"/>
+      </joint>
+      <joint name="rear_right_wheel_joint">
+        <command_interface name="velocity">
+            <param name="min">-15.0</param>
+            <param name="max">15.0</param>
         </command_interface>
         <state_interface name="position"/>

Commit message: update mobo_bot description pkg

File: mobo_bot_description/urdf/four_wheel_base/ros2_control.xacro (robot description, xacro)
@@ -1,20 +1,15 @@
 <?xml version="1.0"?>
 <robot xmlns:xacro="http://www.ros.org/wiki/xacro">
-    <ros2_control name="epmc_hardware_interface" type="system">
+    <ros2_control name="epmc_v2_hardware_interface" type="system">
       <hardware>
-        <plugin>epmc_hardware_interface/EPMC_HardwareInterface</plugin>
+        <plugin>epmc_v2_hardware_interface/EPMC_V2_HardwareInterface</plugin>
         <param name="port">/dev/epmc</param>
-        <param name="motorA_wheel_name">left_wheel_joint</param>
-        <param name="motorB_wheel_name">right_wheel_joint</param>
+        <param name="motor0_wheel_name">front_left_wheel_joint</param>
+        <param name="motor1_wheel_name">front_right_wheel_joint</param>
+        <param name="motor2_wheel_name">rear_left_wheel_joint</param>
+        <param name="motor3_wheel_name">rear_right_wheel_joint</param>
         <param name="cmd_vel_timeout_ms">2000</param>
       </hardware>
-      <!-- <hardware>
-        <plugin>epmc_v2_hardware_interface/EPMC_V2_HardwareInterface</plugin>
-        <param name="port">/dev/epmc</param>
-        <param name="motor0_wheel_name">left_wheel_joint</param>
-        <param name="motor1_wheel_name">right_wheel_joint</param>
-        <param name="cmd_vel_timeout_ms">2000</param>
-      </hardware> -->
-      <joint name="left_wheel_joint">
+      <joint name="front_left_wheel_joint">
         <command_interface name="velocity">
             <param name="min">-15.0</param>
@@ -24,5 +19,21 @@
         <state_interface name="velocity"/>
       </joint>
-      <joint name="right_wheel_joint">
+      <joint name="front_right_wheel_joint">
+        <command_interface name="velocity">
+            <param name="min">-15.0</param>
+            <param name="max">15.0</param>
+        </command_interface>
+        <state_interface name="position"/>
+        <state_interface name="velocity"/>
+      </joint>
+      <joint name="rear_left_wheel_joint">
+        <command_interface name="velocity">
+            <param name="min">-15.0</param>
+            <param name="max">15.0</param>
+        </command_interface>
+        <state_interface name="position"/>
+        <state_interface name="velocity"/>
+      </joint>
+      <joint name="rear_right_wheel_joint">
         <command_interface name="velocity">
             <param name="min">-15.0</param>

File: mobo_bot_description/urdf/two_wheel_base/ros2_control.xacro (robot description, xacro)
@@ -1,15 +1,20 @@
 <?xml version="1.0"?>
 <robot xmlns:xacro="http://www.ros.org/wiki/xacro">
-    <ros2_control name="epmc_v2_hardware_interface" type="system">
+    <ros2_control name="epmc_hardware_interface" type="system">
       <hardware>
+        <plugin>epmc_hardware_interface/EPMC_HardwareInterface</plugin>
+        <param name="port">/dev/epmc</param>
+        <param name="motorA_wheel_name">left_wheel_joint</param>
+        <param name="motorB_wheel_name">right_wheel_joint</param>
+        <param name="cmd_vel_timeout_ms">2000</param>
+      </hardware>
+      <!-- <hardware>
         <plugin>epmc_v2_hardware_interface/EPMC_V2_HardwareInterface</plugin>
         <param name="port">/dev/epmc</param>
-        <param name="motor0_wheel_name">front_left_wheel_joint</param>
-        <param name="motor1_wheel_name">front_right_wheel_joint</param>
-        <param name="motor2_wheel_name">rear_left_wheel_joint</param>
-        <param name="motor3_wheel_name">rear_right_wheel_joint</param>
+        <param name="motor0_wheel_name">left_wheel_joint</param>
+        <param name="motor1_wheel_name">right_wheel_joint</param>
         <param name="cmd_vel_timeout_ms">2000</param>
-      </hardware>
-      <joint name="front_left_wheel_joint">
+      </hardware> -->
+      <joint name="left_wheel_joint">
         <command_interface name="velocity">
             <param name="min">-15.0</param>
@@ -19,21 +24,5 @@
         <state_interface name="velocity"/>
       </joint>
-      <joint name="front_right_wheel_joint">
-        <command_interface name="velocity">
-            <param name="min">-15.0</param>
-            <param name="max">15.0</param>
-        </command_interface>
-        <state_interface name="position"/>
-        <state_interface name="velocity"/>
-      </joint>
-      <joint name="rear_left_wheel_joint">
-        <command_interface name="velocity">
-            <param name="min">-15.0</param>
-            <param name="max">15.0</param>
-        </command_interface>
-        <state_interface name="position"/>
-        <state_interface name="velocity"/>
-      </joint>
-      <joint name="rear_right_wheel_joint">
+      <joint name="right_wheel_joint">
         <command_interface name="velocity">
             <param name="min">-15.0</param>
