Commit message: update mobobot to use new design and hardware

File: mobo_bot_description/urdf/2wheel_base/robot.xacro (robot description, xacro)
@@ -7,16 +7,17 @@
     <xacro:include filename="$(find mobo_bot_description)/urdf/urdf_models/lidar.xacro"/>
     <xacro:include filename="$(find mobo_bot_description)/urdf/urdf_models/cam.xacro"/>
-    <xacro:property name="chassis_length" value="0.22"/>
-    <xacro:property name="chassis_width" value="0.20"/>
+    <xacro:property name="chassis_length" value="0.20"/>
+    <xacro:property name="chassis_width" value="0.18"/>
     <xacro:property name="chassis_height" value="0.05"/>
     <xacro:property name="slab_height" value="0.005"/>
     <xacro:property name="chassis_mass" value="2.0"/>
     <xacro:property name="chassis_color" value="orange"/>
-    <xacro:property name="wheel_seperation" value="0.236"/>
+    <xacro:property name="wheel_seperation" value="0.206"/>
     <xacro:property name="wheel_radius" value="0.034"/>
-    <xacro:property name="wheel_width" value="0.026"/>
+    <xacro:property name="wheel_width" value="0.015"/>
     <xacro:property name="wheel_mass" value="0.08"/>
-    <xacro:property name="wheel_height_offset" value="0.025"/>
-    <xacro:property name="wheel_base_dist" value="0.12"/>
+    <xacro:property name="wheel_height_offset" value="0.01"/>
+    <xacro:property name="castor_wheel_diameter" value="${wheel_radius+wheel_height_offset}"/>
+    <xacro:property name="castor_wheel_mass" value="0.08"/>
     <link name="base_link">
     </link>
@@ -27,12 +28,12 @@
     </joint>
     <link name="chassis">
-        <xacro:insert_box_with_fillet x="0" y="0" z="0"
+        <xacro:insert_box_with_fillet x="-0.040" y="0" z="0"
             size_x="${chassis_length}" size_y="${chassis_width}" size_z="${slab_height}"
-            fillet_radius="0.025"/>
-        <xacro:insert_box_with_fillet x="0" y="0" z="${chassis_height}"
+            fillet_radius="0.02"/>
+        <xacro:insert_box_with_fillet x="-0.040" y="0" z="${chassis_height}"
             size_x="${chassis_length}" size_y="${chassis_width}" size_z="${slab_height}"
             fillet_radius="0.02"/>
         <visual>
-            <origin xyz="0.09 0.08 ${chassis_height/2}" rpy="0 0 0"/>
+            <origin xyz="0.04 0.07 ${chassis_height/2}" rpy="0 0 0"/>
             <geometry>
                 <cylinder radius="0.004" length="${chassis_height}"/>
@@ -41,5 +42,5 @@
         </visual>
         <visual>
-            <origin xyz="0.09 -0.08 ${chassis_height/2}" rpy="0 0 0"/>
+            <origin xyz="0.04 -0.07 ${chassis_height/2}" rpy="0 0 0"/>
             <geometry>
                 <cylinder radius="0.004" length="${chassis_height}"/>
@@ -48,5 +49,5 @@
         </visual>
         <visual>
-            <origin xyz="-0.09 0.08 ${chassis_height/2}" rpy="0 0 0"/>
+            <origin xyz="-0.12 0.07 ${chassis_height/2}" rpy="0 0 0"/>
             <geometry>
                 <cylinder radius="0.004" length="${chassis_height}"/>
@@ -55,5 +56,5 @@
         </visual>
         <visual>
-            <origin xyz="-0.09 -0.08 ${chassis_height/2}" rpy="0 0 0"/>
+            <origin xyz="-0.12 -0.07 ${chassis_height/2}" rpy="0 0 0"/>
             <geometry>
                 <cylinder radius="0.004" length="${chassis_height}"/>
@@ -62,5 +63,5 @@
         </visual>
         <collision>
-           <origin xyz="0 0 ${chassis_height/2}" rpy="0 0 0"/>
+           <origin xyz="-0.04 0 ${chassis_height/2}" rpy="0 0 0"/>
             <geometry>
                 <box size="${chassis_length} ${chassis_width} ${chassis_height}"/>
@@ -68,69 +69,68 @@
         </collision>
         <xacro:inertial_box mass="${chassis_mass}" x="${chassis_length}" y="${chassis_width}" z="${chassis_height}">
-            <origin xyz="0 0 ${chassis_height/2}" rpy="0 0 0"/>
+            <origin xyz="-0.07 0 ${chassis_height/2}" rpy="0 0 0"/>
         </xacro:inertial_box>
     </link>
     <xacro:insert_drive_wheel
-        base_name="front_left_wheel"
+        base_name="left_wheel"
         parent_name="base_link"
-        x="${wheel_base_dist/2}" y="${wheel_seperation/2}" z="${wheel_radius}"
+        x="0" y="${wheel_seperation/2}" z="${wheel_radius}"
         mass="${wheel_mass}"
         radius="${wheel_radius}"
         thickness="${wheel_width}"/>
     <xacro:insert_drive_wheel_rim
-        base_name="front_left_rim"
-        parent_name="front_left_wheel"
+        base_name="left_rim"
+        parent_name="left_wheel"
         radius="${wheel_radius}"
         thickness="${wheel_width}"
         spoke_width="0.005"/>
     <xacro:insert_drive_wheel
-        base_name="front_right_wheel"
+        base_name="right_wheel"
         parent_name="base_link"
-        x="${wheel_base_dist/2}" y="${-wheel_seperation/2}" z="${wheel_radius}"
+        x="0" y="${-wheel_seperation/2}" z="${wheel_radius}"
         mass="${wheel_mass}"
         radius="${wheel_radius}"
         thickness="${wheel_width}"/>
     <xacro:insert_drive_wheel_rim
-        base_name="front_right_rim"
-        parent_name="front_right_wheel"
+        base_name="right_rim"
+        parent_name="right_wheel"
         radius="${wheel_radius}"
         thickness="${wheel_width}"
         spoke_width="0.005"/>
-    <xacro:insert_drive_wheel
-        base_name="rear_left_wheel"
-        parent_name="base_link"
-        x="${-wheel_base_dist/2}" y="${wheel_seperation/2}" z="${wheel_radius}"
-        mass="${wheel_mass}"
-        radius="${wheel_radius}"
-        thickness="${wheel_width}"/>
-    <xacro:insert_drive_wheel_rim
-        base_name="rear_left_rim"
-        parent_name="rear_left_wheel"
-        radius="${wheel_radius}"
-        thickness="${wheel_width}"
-        spoke_width="0.005"/>
-    <xacro:insert_drive_wheel
-        base_name="rear_right_wheel"
-        parent_name="base_link"
-        x="${-wheel_base_dist/2}" y="${-wheel_seperation/2}" z="${wheel_radius}"
-        mass="${wheel_mass}"
-        radius="${wheel_radius}"
-        thickness="${wheel_width}"/>
-    <xacro:insert_drive_wheel_rim
-        base_name="rear_right_rim"
-        parent_name="rear_right_wheel"
-        radius="${wheel_radius}"
-        thickness="${wheel_width}"
-        spoke_width="0.005"/>
+    <joint name="castor_wheel_joint" type="fixed">
+        <parent link="base_link"/>
+        <child link="castor_wheel"/>
+        <origin xyz="-0.10 0 ${castor_wheel_diameter/2}"/>
+    </joint>
+    <link name="castor_wheel">
+        <visual>
+            <origin xyz="0 0 0" rpy="0 0 0"/>
+            <geometry>
+                <sphere radius="${castor_wheel_diameter/2}" />
+            </geometry>
+            <material name="grey">
+                <color rgba="0.25 0.25 0.25 1"/>
+            </material>
+        </visual>
+        <collision>
+           <origin xyz="0 0 0" rpy="0 0 0"/>
+            <geometry>
+                <sphere radius="${castor_wheel_diameter/2}" />
+            </geometry>
+        </collision>
+        <xacro:inertial_sphere mass="${castor_wheel_mass}" radius="${castor_wheel_diameter/2}">
+            <origin xyz="0 0 0" rpy="0 0 0"/>
+        </xacro:inertial_sphere>
+    </link>
     <xacro:property name="lidar_z_offset" value="0.04"/>
     <xacro:insert_lidar
         base_name="lidar"
         parent_name="chassis"
-        x="0.05" y="0" z="${chassis_height+lidar_z_offset}"
+        x="-0.0115" y="0" z="${chassis_height+lidar_z_offset}"
         mass="0.1"/>
     <joint name="imu_joint" type="fixed">
         <parent link="chassis"/>
         <child link="imu"/>
-        <origin xyz="0 0 ${slab_height}"/>
+        <origin xyz="0.03 0 ${chassis_height}"/>
     </joint>
     <link name="imu"></link>
@@ -138,10 +138,10 @@
         base_name="sonar"
         parent_name="chassis"
-        x="0.11" y="0" z="${chassis_height/6}"
+        x="0.07" y="0" z="${chassis_height/6}"
         mass="0.005"/>
     <xacro:insert_camera
         base_name="camera"
         parent_name="chassis"
-        x="0.13" y="0" z="${chassis_height+0.015}"
+        x="0.09" y="0" z="${chassis_height+0.015}"
         mass="0.005" tilt_angle="0.00"/>
 </robot>

File: mobo_bot_description/urdf/2wheel_base/ros2_control.xacro (robot description, xacro)
@@ -4,31 +4,24 @@
       <hardware>
         <plugin>epmc_hardware_interface/EPMC_HardwareInterface</plugin>
-        <param name="port">/dev/epmc</param>
-        <param name="motorA_wheel_name">left_wheel_joint</param>
-        <param name="motorB_wheel_name">right_wheel_joint</param>
-        <param name="cmd_vel_timeout_ms">2000</param>
-      </hardware>
-      <!-- <hardware>
-        <plugin>epmc_v2_hardware_interface/EPMC_V2_HardwareInterface</plugin>
-        <param name="port">/dev/epmc</param>
+        <param name="serial_port">/dev/epmc</param>
+        <param name="serial_baud_rate">115200</param>
+        <param name="serial_timeout_ms">16</param>
         <param name="motor0_wheel_name">left_wheel_joint</param>
         <param name="motor1_wheel_name">right_wheel_joint</param>
         <param name="cmd_vel_timeout_ms">2000</param>
-      </hardware> -->
+      </hardware>
       <joint name="left_wheel_joint">
         <command_interface name="velocity">
-            <param name="min">-15.0</param>
-            <param name="max">15.0</param>
+            <param name="min">-8.0</param>
+            <param name="max">8.0</param>
         </command_interface>
         <state_interface name="position"/>
-        <state_interface name="velocity"/>
       </joint>
       <joint name="right_wheel_joint">
         <command_interface name="velocity">
-            <param name="min">-15.0</param>
-            <param name="max">15.0</param>
+            <param name="min">-8.0</param>
+            <param name="max">8.0</param>
         </command_interface>
         <state_interface name="position"/>
-        <state_interface name="velocity"/>
       </joint>
     </ros2_control>

File: mobo_bot_description/urdf/4wheel_std_base/robot.xacro (robot description, xacro)
@@ -7,5 +7,5 @@
     <xacro:include filename="$(find mobo_bot_description)/urdf/urdf_models/lidar.xacro"/>
     <xacro:include filename="$(find mobo_bot_description)/urdf/urdf_models/cam.xacro"/>
-    <xacro:property name="chassis_length" value="0.22"/>
+    <xacro:property name="chassis_length" value="0.24"/>
     <xacro:property name="chassis_width" value="0.20"/>
     <xacro:property name="chassis_height" value="0.05"/>
@@ -18,6 +18,5 @@
     <xacro:property name="wheel_mass" value="0.08"/>
     <xacro:property name="wheel_height_offset" value="0.025"/>
-    <xacro:property name="castor_wheel_diameter" value="${wheel_radius+wheel_height_offset}"/>
-    <xacro:property name="castor_wheel_mass" value="0.08"/>
+    <xacro:property name="wheel_base_dist" value="0.12"/>
     <link name="base_link">
     </link>
@@ -28,12 +27,12 @@
     </joint>
     <link name="chassis">
-        <xacro:insert_box_with_fillet x="-0.040" y="0" z="0"
+        <xacro:insert_box_with_fillet x="0" y="0" z="0"
             size_x="${chassis_length}" size_y="${chassis_width}" size_z="${slab_height}"
-            fillet_radius="0.02"/>
-        <xacro:insert_box_with_fillet x="-0.040" y="0" z="${chassis_height}"
+            fillet_radius="0.025"/>
+        <xacro:insert_box_with_fillet x="0" y="0" z="${chassis_height}"
             size_x="${chassis_length}" size_y="${chassis_width}" size_z="${slab_height}"
             fillet_radius="0.02"/>
         <visual>
-            <origin xyz="0.05 0.08 ${chassis_height/2}" rpy="0 0 0"/>
+            <origin xyz="0.1 0.08 ${chassis_height/2}" rpy="0 0 0"/>
             <geometry>
                 <cylinder radius="0.004" length="${chassis_height}"/>
@@ -42,5 +41,5 @@
         </visual>
         <visual>
-            <origin xyz="0.05 -0.08 ${chassis_height/2}" rpy="0 0 0"/>
+            <origin xyz="0.1 -0.08 ${chassis_height/2}" rpy="0 0 0"/>
             <geometry>
                 <cylinder radius="0.004" length="${chassis_height}"/>
@@ -49,5 +48,5 @@
         </visual>
         <visual>
-            <origin xyz="-0.13 0.08 ${chassis_height/2}" rpy="0 0 0"/>
+            <origin xyz="-0.1 0.08 ${chassis_height/2}" rpy="0 0 0"/>
             <geometry>
                 <cylinder radius="0.004" length="${chassis_height}"/>
@@ -56,5 +55,5 @@
         </visual>
         <visual>
-            <origin xyz="-0.13 -0.08 ${chassis_height/2}" rpy="0 0 0"/>
+            <origin xyz="-0.1 -0.08 ${chassis_height/2}" rpy="0 0 0"/>
             <geometry>
                 <cylinder radius="0.004" length="${chassis_height}"/>
@@ -63,5 +62,5 @@
         </visual>
         <collision>
-           <origin xyz="-0.04 0 ${chassis_height/2}" rpy="0 0 0"/>
+           <origin xyz="0 0 ${chassis_height/2}" rpy="0 0 0"/>
             <geometry>
                 <box size="${chassis_length} ${chassis_width} ${chassis_height}"/>
@@ -69,68 +68,69 @@
         </collision>
         <xacro:inertial_box mass="${chassis_mass}" x="${chassis_length}" y="${chassis_width}" z="${chassis_height}">
-            <origin xyz="-0.07 0 ${chassis_height/2}" rpy="0 0 0"/>
+            <origin xyz="0 0 ${chassis_height/2}" rpy="0 0 0"/>
         </xacro:inertial_box>
     </link>
     <xacro:insert_drive_wheel
-        base_name="left_wheel"
+        base_name="front_left_wheel"
         parent_name="base_link"
-        x="0" y="${wheel_seperation/2}" z="${wheel_radius}"
+        x="${wheel_base_dist/2}" y="${wheel_seperation/2}" z="${wheel_radius}"
         mass="${wheel_mass}"
         radius="${wheel_radius}"
         thickness="${wheel_width}"/>
     <xacro:insert_drive_wheel_rim
-        base_name="left_rim"
-        parent_name="left_wheel"
+        base_name="front_left_rim"
+        parent_name="front_left_wheel"
         radius="${wheel_radius}"
         thickness="${wheel_width}"
         spoke_width="0.005"/>
     <xacro:insert_drive_wheel
-        base_name="right_wheel"
+        base_name="front_right_wheel"
         parent_name="base_link"
-        x="0" y="${-wheel_seperation/2}" z="${wheel_radius}"
+        x="${wheel_base_dist/2}" y="${-wheel_seperation/2}" z="${wheel_radius}"
         mass="${wheel_mass}"
         radius="${wheel_radius}"
         thickness="${wheel_width}"/>
     <xacro:insert_drive_wheel_rim
-        base_name="right_rim"
-        parent_name="right_wheel"
+        base_name="front_right_rim"
+        parent_name="front_right_wheel"
         radius="${wheel_radius}"
         thickness="${wheel_width}"
         spoke_width="0.005"/>
-    <joint name="castor_wheel_joint" type="fixed">
-        <parent link="base_link"/>
-        <child link="castor_wheel"/>
-        <origin xyz="-0.10 0 ${castor_wheel_diameter/2}"/>
-    </joint>
-    <link name="castor_wheel">
-        <visual>
-            <origin xyz="0 0 0" rpy="0 0 0"/>
-            <geometry>
-                <sphere radius="${castor_wheel_diameter/2}" />
-            </geometry>
-            <material name="grey">
-                <color rgba="0.25 0.25 0.25 1"/>
-            </material>
-        </visual>
-        <collision>
-           <origin xyz="0 0 0" rpy="0 0 0"/>
-            <geometry>
-                <sphere radius="${castor_wheel_diameter/2}" />
-            </geometry>
-        </collision>
-        <xacro:inertial_sphere mass="${castor_wheel_mass}" radius="${castor_wheel_diameter/2}">
-            <origin xyz="0 0 0" rpy="0 0 0"/>
-        </xacro:inertial_sphere>
-    </link>
+    <xacro:insert_drive_wheel
+        base_name="rear_left_wheel"
+        parent_name="base_link"
+        x="${-wheel_base_dist/2}" y="${wheel_seperation/2}" z="${wheel_radius}"
+        mass="${wheel_mass}"
+        radius="${wheel_radius}"
+        thickness="${wheel_width}"/>
+    <xacro:insert_drive_wheel_rim
+        base_name="rear_left_rim"
+        parent_name="rear_left_wheel"
+        radius="${wheel_radius}"
+        thickness="${wheel_width}"
+        spoke_width="0.005"/>
+    <xacro:insert_drive_wheel
+        base_name="rear_right_wheel"
+        parent_name="base_link"
+        x="${-wheel_base_dist/2}" y="${-wheel_seperation/2}" z="${wheel_radius}"
+        mass="${wheel_mass}"
+        radius="${wheel_radius}"
+        thickness="${wheel_width}"/>
+    <xacro:insert_drive_wheel_rim
+        base_name="rear_right_rim"
+        parent_name="rear_right_wheel"
+        radius="${wheel_radius}"
+        thickness="${wheel_width}"
+        spoke_width="0.005"/>
     <xacro:property name="lidar_z_offset" value="0.04"/>
     <xacro:insert_lidar
         base_name="lidar"
         parent_name="chassis"
-        x="0.01" y="0" z="${chassis_height+lidar_z_offset}"
+        x="0.05" y="0" z="${chassis_height+lidar_z_offset}"
         mass="0.1"/>
     <joint name="imu_joint" type="fixed">
         <parent link="chassis"/>
         <child link="imu"/>
-        <origin xyz="0 0 ${chassis_height}"/>
+        <origin xyz="0 0 ${slab_height}"/>
     </joint>
     <link name="imu"></link>
@@ -138,10 +138,10 @@
         base_name="sonar"
         parent_name="chassis"
-        x="0.07" y="0" z="${chassis_height/6}"
+        x="0.11" y="0" z="${chassis_height/6}"
         mass="0.005"/>
     <xacro:insert_camera
         base_name="camera"
         parent_name="chassis"
-        x="0.09" y="0" z="${chassis_height+0.015}"
+        x="0.13" y="0" z="${chassis_height+0.015}"
         mass="0.005" tilt_angle="0.00"/>
 </robot>

File: mobo_bot_description/urdf/robot_urdf.xacro (robot description, xacro)
@@ -2,6 +2,6 @@
 <robot name="mobo_bot" xmlns:xacro="http://www.ros.org/wiki/xacro">
     <xacro:arg name="run_gz_sim" default="false"/>
-    <xacro:arg name="wheel_type" default="2wheel"/>
-    <xacro:property name="wheel_type_name" value="$(arg wheel_type)"/>
+    <xacro:arg name="base_type" default="2WHEEL"/>
+    <xacro:property name="MOBOBOT_BASE_TYPE" value="$(arg base_type)"/>
     <material name="orange">
         <color rgba="1 0.55 0 1"/>
@@ -50,20 +50,29 @@
     </xacro:macro>
     <!-- Conditional inclusion -->
-    <xacro:if value="${wheel_type_name == '4wheel'}">
-        <xacro:include filename="$(find mobo_bot_description)/urdf/four_wheel_base/robot.xacro" />
+    <xacro:if value="${MOBOBOT_BASE_TYPE == '2WHEEL'}">
+        <xacro:include filename="$(find mobo_bot_description)/urdf/2wheel_base/robot.xacro" />
         <xacro:if value="$(arg run_gz_sim)">
-            <xacro:include filename="$(find mobo_bot_description)/urdf/four_wheel_base/gazebo_properties.xacro" />
+            <xacro:include filename="$(find mobo_bot_description)/urdf/2wheel_base/gazebo_properties.xacro" />
         </xacro:if>
         <xacro:unless value="$(arg run_gz_sim)">
-            <xacro:include filename="$(find mobo_bot_description)/urdf/four_wheel_base/ros2_control.xacro" />
+            <xacro:include filename="$(find mobo_bot_description)/urdf/2wheel_base/ros2_control.xacro" />
         </xacro:unless>
     </xacro:if>
-    <xacro:if value="${wheel_type_name == '2wheel'}">
-        <xacro:include filename="$(find mobo_bot_description)/urdf/two_wheel_base/robot.xacro" />
+    <xacro:if value="${MOBOBOT_BASE_TYPE == '2WHEEL_STD'}">
+        <xacro:include filename="$(find mobo_bot_description)/urdf/2wheel_std_base/robot.xacro" />
         <xacro:if value="$(arg run_gz_sim)">
-            <xacro:include filename="$(find mobo_bot_description)/urdf/two_wheel_base/gazebo_properties.xacro" />
+            <xacro:include filename="$(find mobo_bot_description)/urdf/2wheel_std_base/gazebo_properties.xacro" />
         </xacro:if>
         <xacro:unless value="$(arg run_gz_sim)">
-            <xacro:include filename="$(find mobo_bot_description)/urdf/two_wheel_base/ros2_control.xacro" />
+            <xacro:include filename="$(find mobo_bot_description)/urdf/2wheel_std_base/ros2_control.xacro" />
+        </xacro:unless>
+    </xacro:if>
+    <xacro:if value="${MOBOBOT_BASE_TYPE == '4WHEEL_STD'}">
+        <xacro:include filename="$(find mobo_bot_description)/urdf/4wheel_std_base/robot.xacro" />
+        <xacro:if value="$(arg run_gz_sim)">
+            <xacro:include filename="$(find mobo_bot_description)/urdf/4wheel_std_base/gazebo_properties.xacro" />
+        </xacro:if>
+        <xacro:unless value="$(arg run_gz_sim)">
+            <xacro:include filename="$(find mobo_bot_description)/urdf/4wheel_std_base/ros2_control.xacro" />
         </xacro:unless>
     </xacro:if>
