Commit message: full update for mecanum wheel

File: mobo_bot_description/urdf/22WD/robot.xacro (robot description, xacro)
@@ -7,15 +7,15 @@
     <xacro:include filename="$(find mobo_bot_description)/urdf/urdf_models/lidar.xacro"/>
     <xacro:include filename="$(find mobo_bot_description)/urdf/urdf_models/cam.xacro"/>
-    <xacro:property name="chassis_length" value="0.20"/>
-    <xacro:property name="chassis_width" value="0.18"/>
+    <xacro:property name="chassis_length" value="0.24"/>
+    <xacro:property name="chassis_width" value="0.20"/>
     <xacro:property name="chassis_height" value="0.05"/>
     <xacro:property name="slab_height" value="0.005"/>
     <xacro:property name="chassis_mass" value="2.0"/>
     <xacro:property name="chassis_color" value="orange"/>
-    <xacro:property name="wheel_seperation" value="0.206"/>
+    <xacro:property name="wheel_seperation" value="0.236"/>
     <xacro:property name="wheel_radius" value="0.034"/>
-    <xacro:property name="wheel_width" value="0.015"/>
+    <xacro:property name="wheel_width" value="0.026"/>
     <xacro:property name="wheel_mass" value="0.08"/>
-    <xacro:property name="wheel_height_offset" value="0.01"/>
+    <xacro:property name="wheel_height_offset" value="0.025"/>
     <xacro:property name="castor_wheel_diameter" value="${wheel_radius+wheel_height_offset}"/>
     <xacro:property name="castor_wheel_mass" value="0.08"/>
@@ -35,5 +35,5 @@
             fillet_radius="0.02"/>
         <visual>
-            <origin xyz="0.04 0.07 ${chassis_height/2}" rpy="0 0 0"/>
+            <origin xyz="0.06 0.08 ${chassis_height/2}" rpy="0 0 0"/>
             <geometry>
                 <cylinder radius="0.004" length="${chassis_height}"/>
@@ -42,5 +42,5 @@
         </visual>
         <visual>
-            <origin xyz="0.04 -0.07 ${chassis_height/2}" rpy="0 0 0"/>
+            <origin xyz="0.06 -0.08 ${chassis_height/2}" rpy="0 0 0"/>
             <geometry>
                 <cylinder radius="0.004" length="${chassis_height}"/>
@@ -49,5 +49,5 @@
         </visual>
         <visual>
-            <origin xyz="-0.12 0.07 ${chassis_height/2}" rpy="0 0 0"/>
+            <origin xyz="-0.14 0.08 ${chassis_height/2}" rpy="0 0 0"/>
             <geometry>
                 <cylinder radius="0.004" length="${chassis_height}"/>
@@ -56,5 +56,5 @@
         </visual>
         <visual>
-            <origin xyz="-0.12 -0.07 ${chassis_height/2}" rpy="0 0 0"/>
+            <origin xyz="-0.14 -0.08 ${chassis_height/2}" rpy="0 0 0"/>
             <geometry>
                 <cylinder radius="0.004" length="${chassis_height}"/>
@@ -101,5 +101,5 @@
         <parent link="base_link"/>
         <child link="castor_wheel"/>
-        <origin xyz="-0.10 0 ${castor_wheel_diameter/2}"/>
+        <origin xyz="-0.11 0 ${castor_wheel_diameter/2}"/>
     </joint>
     <link name="castor_wheel">
@@ -123,21 +123,21 @@
         </xacro:inertial_sphere>
     </link>
+    <xacro:insert_sonar
+        base_name="sonar"
+        parent_name="chassis"
+        x="0.08" y="0" z="${chassis_height/6}"
+        mass="0.005"/>
     <xacro:property name="lidar_z_offset" value="0.04"/>
     <xacro:insert_lidar
         base_name="lidar"
         parent_name="chassis"
-        x="-0.0115" y="0" z="${chassis_height+lidar_z_offset}"
+        x="0.01" y="0" z="${chassis_height+lidar_z_offset}"
         mass="0.1"/>
     <joint name="imu_joint" type="fixed">
         <parent link="chassis"/>
         <child link="imu"/>
-        <origin xyz="0.03 0 ${chassis_height}"/>
+        <origin xyz="0 0 ${chassis_height}"/>
     </joint>
     <link name="imu"></link>
-    <xacro:insert_sonar
-        base_name="sonar"
-        parent_name="chassis"
-        x="0.07" y="0" z="${chassis_height/6}"
-        mass="0.005"/>
     <xacro:insert_camera
         base_name="camera"

File: mobo_bot_description/urdf/2WD/robot.xacro (robot description, xacro)
@@ -7,15 +7,15 @@
     <xacro:include filename="$(find mobo_bot_description)/urdf/urdf_models/lidar.xacro"/>
     <xacro:include filename="$(find mobo_bot_description)/urdf/urdf_models/cam.xacro"/>
-    <xacro:property name="chassis_length" value="0.24"/>
-    <xacro:property name="chassis_width" value="0.20"/>
+    <xacro:property name="chassis_length" value="0.20"/>
+    <xacro:property name="chassis_width" value="0.18"/>
     <xacro:property name="chassis_height" value="0.05"/>
     <xacro:property name="slab_height" value="0.005"/>
     <xacro:property name="chassis_mass" value="2.0"/>
     <xacro:property name="chassis_color" value="orange"/>
-    <xacro:property name="wheel_seperation" value="0.236"/>
-    <xacro:property name="wheel_radius" value="0.034"/>
-    <xacro:property name="wheel_width" value="0.026"/>
+    <xacro:property name="wheel_seperation" value="0.207"/>
+    <xacro:property name="wheel_radius" value="0.033"/>
+    <xacro:property name="wheel_width" value="0.015"/>
     <xacro:property name="wheel_mass" value="0.08"/>
-    <xacro:property name="wheel_height_offset" value="0.025"/>
+    <xacro:property name="wheel_height_offset" value="0.01"/>
     <xacro:property name="castor_wheel_diameter" value="${wheel_radius+wheel_height_offset}"/>
     <xacro:property name="castor_wheel_mass" value="0.08"/>
@@ -35,5 +35,5 @@
             fillet_radius="0.02"/>
         <visual>
-            <origin xyz="0.06 0.08 ${chassis_height/2}" rpy="0 0 0"/>
+            <origin xyz="0.04 0.07 ${chassis_height/2}" rpy="0 0 0"/>
             <geometry>
                 <cylinder radius="0.004" length="${chassis_height}"/>
@@ -42,5 +42,5 @@
         </visual>
         <visual>
-            <origin xyz="0.06 -0.08 ${chassis_height/2}" rpy="0 0 0"/>
+            <origin xyz="0.04 -0.07 ${chassis_height/2}" rpy="0 0 0"/>
             <geometry>
                 <cylinder radius="0.004" length="${chassis_height}"/>
@@ -49,5 +49,5 @@
         </visual>
         <visual>
-            <origin xyz="-0.14 0.08 ${chassis_height/2}" rpy="0 0 0"/>
+            <origin xyz="-0.12 0.07 ${chassis_height/2}" rpy="0 0 0"/>
             <geometry>
                 <cylinder radius="0.004" length="${chassis_height}"/>
@@ -56,5 +56,5 @@
         </visual>
         <visual>
-            <origin xyz="-0.14 -0.08 ${chassis_height/2}" rpy="0 0 0"/>
+            <origin xyz="-0.12 -0.07 ${chassis_height/2}" rpy="0 0 0"/>
             <geometry>
                 <cylinder radius="0.004" length="${chassis_height}"/>
@@ -101,5 +101,5 @@
         <parent link="base_link"/>
         <child link="castor_wheel"/>
-        <origin xyz="-0.11 0 ${castor_wheel_diameter/2}"/>
+        <origin xyz="-0.10 0 ${castor_wheel_diameter/2}"/>
     </joint>
     <link name="castor_wheel">
@@ -123,21 +123,21 @@
         </xacro:inertial_sphere>
     </link>
+    <xacro:insert_sonar
+        base_name="sonar"
+        parent_name="chassis"
+        x="0.055" y="0" z="${chassis_height/6}"
+        mass="0.005"/>
     <xacro:property name="lidar_z_offset" value="0.04"/>
     <xacro:insert_lidar
         base_name="lidar"
         parent_name="chassis"
-        x="0.01" y="0" z="${chassis_height+lidar_z_offset}"
+        x="-0.0115" y="0" z="${chassis_height+lidar_z_offset}"
         mass="0.1"/>
     <joint name="imu_joint" type="fixed">
         <parent link="chassis"/>
         <child link="imu"/>
-        <origin xyz="0 0 ${chassis_height}"/>
+        <origin xyz="0.03 0 ${chassis_height}"/>
     </joint>
     <link name="imu"></link>
-    <xacro:insert_sonar
-        base_name="sonar"
-        parent_name="chassis"
-        x="0.07" y="0" z="${chassis_height/6}"
-        mass="0.005"/>
     <xacro:insert_camera
         base_name="camera"

File: mobo_bot_description/urdf/MEC/robot.xacro (robot description, xacro)
@@ -2,6 +2,5 @@
 <robot name="mobo_bot" xmlns:xacro="http://www.ros.org/wiki/xacro">
     <xacro:include filename="$(find mobo_bot_description)/urdf/urdf_models/box_with_fillet_macro.xacro"/>
-    <xacro:include filename="$(find mobo_bot_description)/urdf/urdf_models/drive_wheel_macro.xacro"/>
-    <xacro:include filename="$(find mobo_bot_description)/urdf/urdf_models/drive_wheel_rim_macro.xacro"/>
+    <xacro:include filename="$(find mobo_bot_description)/urdf/urdf_models/mecanum_drive_wheel_macro.xacro"/>
     <xacro:include filename="$(find mobo_bot_description)/urdf/urdf_models/sonar.xacro"/>
     <xacro:include filename="$(find mobo_bot_description)/urdf/urdf_models/lidar.xacro"/>
@@ -71,5 +70,5 @@
         </xacro:inertial_box>
     </link>
-    <xacro:insert_drive_wheel
+    <xacro:insert_mecanum_left_wheel
         base_name="front_left_wheel"
         parent_name="base_link"
@@ -78,11 +77,5 @@
         radius="${wheel_radius}"
         thickness="${wheel_width}"/>
-    <xacro:insert_drive_wheel_rim
-        base_name="front_left_rim"
-        parent_name="front_left_wheel"
-        radius="${wheel_radius}"
-        thickness="${wheel_width}"
-        spoke_width="0.005"/>
-    <xacro:insert_drive_wheel
+    <xacro:insert_mecanum_right_wheel
         base_name="front_right_wheel"
         parent_name="base_link"
@@ -91,11 +84,5 @@
         radius="${wheel_radius}"
         thickness="${wheel_width}"/>
-    <xacro:insert_drive_wheel_rim
-        base_name="front_right_rim"
-        parent_name="front_right_wheel"
-        radius="${wheel_radius}"
-        thickness="${wheel_width}"
-        spoke_width="0.005"/>
-    <xacro:insert_drive_wheel
+    <xacro:insert_mecanum_left_wheel
         base_name="rear_left_wheel"
         parent_name="base_link"
@@ -104,11 +91,5 @@
         radius="${wheel_radius}"
         thickness="${wheel_width}"/>
-    <xacro:insert_drive_wheel_rim
-        base_name="rear_left_rim"
-        parent_name="rear_left_wheel"
-        radius="${wheel_radius}"
-        thickness="${wheel_width}"
-        spoke_width="0.005"/>
-    <xacro:insert_drive_wheel
+    <xacro:insert_mecanum_right_wheel
         base_name="rear_right_wheel"
         parent_name="base_link"
@@ -117,10 +98,9 @@
         radius="${wheel_radius}"
         thickness="${wheel_width}"/>
-    <xacro:insert_drive_wheel_rim
-        base_name="rear_right_rim"
-        parent_name="rear_right_wheel"
-        radius="${wheel_radius}"
-        thickness="${wheel_width}"
-        spoke_width="0.005"/>
+    <xacro:insert_sonar
+        base_name="sonar"
+        parent_name="chassis"
+        x="0.12" y="0" z="${chassis_height/6}"
+        mass="0.005"/>
     <xacro:property name="lidar_z_offset" value="0.04"/>
     <xacro:insert_lidar
@@ -135,9 +115,4 @@
     </joint>
     <link name="imu"></link>
-    <xacro:insert_sonar
-        base_name="sonar"
-        parent_name="chassis"
-        x="0.11" y="0" z="${chassis_height/6}"
-        mass="0.005"/>
     <xacro:insert_camera
         base_name="camera"

File: mobo_bot_description/urdf/robot_gazebo_properties.xacro (robot description, xacro)
@@ -1,4 +1,4 @@
 <?xml version="1.0"?>
-<robot xmlns:xacro="http://ros.org/wiki/xacro">
+<robot xmlns:xacro="http://www.ros.org/wiki/xacro" xmlns:gz="http://gazebosim.org/schema">
   <xacro:macro name="gz_material_orange">
     <material>
@@ -49,48 +49,46 @@
     </material>
   </xacro:macro>
-  <gazebo reference="chassis">
+  <gazebo reference="sonar">
     <visual>
-      <xacro:gz_material_orange/>
+      <xacro:gz_material_blue/>
     </visual>
   </gazebo>
-  <gazebo reference="left_wheel">
+  <gazebo reference="lidar">
     <visual>
-      <xacro:gz_material_black/>
+      <xacro:gz_material_grey/>
     </visual>
-    <mu1>1.0</mu1>
-    <mu2>1.0</mu2>
+    <sensor name="lidar" type="gpu_lidar">
+      <topic>lidar/scan</topic>
+      <gz_frame_id>lidar</gz_frame_id>
+      <always_on>true</always_on>
+      <visualize>true</visualize>
+      <update_rate>10.0</update_rate>
+      <ray>
+        <scan>
+          <horizontal>
+            <samples>360</samples>
+            <min_angle>${-0.833*pi}</min_angle>
+            <max_angle>${0.833*pi}</max_angle>
+            <resolution>1</resolution>
+          </horizontal>
+        </scan>
+        <range>
+          <min>0.1</min>
+          <max>10.0</max>
+          <resolution>0.01</resolution>
+        </range>
+        <noise>
+          <type>gaussian</type>
+          <mean>0.0</mean>
+          <stddev>0.01</stddev>
+        </noise>
+      </ray>
+    </sensor>
   </gazebo>
-  <gazebo reference="left_rim">
-    <visual>
-      <xacro:gz_material_red/>
-    </visual>
-  </gazebo>
-  <gazebo reference="right_wheel">
-    <visual>
-      <xacro:gz_material_black/>
-    </visual>
-    <mu1>1.0</mu1>
-    <mu2>1.0</mu2>
-  </gazebo>
-  <gazebo reference="right_rim">
-    <visual>
-      <xacro:gz_material_red/>
-    </visual>
-  </gazebo>
-  <gazebo reference="castor_wheel">
-    <visual>
-      <xacro:gz_material_silver/>
-    </visual>
-    <mu1>0.001</mu1>
-    <mu2>0.001</mu2>
-  </gazebo>
-  <!-- <gazebo reference="imu">
+  <gazebo reference="imu">
     <sensor name="imu" type="imu">
-      <ignition_frame_id>imu</ignition_frame_id>
-      <plugin filename="ignition-gazebo-imu-system" name="ignition::gazebo::systems::Imu">
-      </plugin>
       <topic>imu/data</topic>
       <always_on>true</always_on>
-      <update_rate>10</update_rate>
+      <update_rate>50</update_rate>
       <visualize>true</visualize>
       <imu>
@@ -149,40 +147,4 @@
       </imu>
     </sensor>
-  </gazebo> -->
-  <gazebo reference="sonar">
-    <visual>
-      <xacro:gz_material_blue/>
-    </visual>
-  </gazebo>
-  <gazebo reference="lidar">
-    <visual>
-      <xacro:gz_material_grey/>
-    </visual>
-    <sensor name="lidar" type="gpu_lidar">
-      <gz_frame_id>lidar</gz_frame_id>
-      <ray>
-        <scan>
-          <horizontal>
-            <samples>360</samples>
-            <min_angle>${-0.833*pi}</min_angle>
-            <max_angle>${0.833*pi}</max_angle>
-            <resolution>1</resolution>
-          </horizontal>
-        </scan>
-        <range>
-          <min>0.1</min>
-          <max>8.0</max>
-          <resolution>0.01</resolution>
-        </range>
-        <noise>
-          <type>gaussian</type>
-          <mean>0.0</mean>
-          <stddev>0.01</stddev>
-        </noise>
-      </ray>
-      <always_on>true</always_on>
-      <visualize>true</visualize>
-      <update_rate>10.0</update_rate>
-    </sensor>
   </gazebo>
   <gazebo reference="camera">
@@ -192,60 +154,24 @@
     <sensor name="camera_optical" type="camera">
     <!-- <sensor name="camera_optical" type="depth"> -->
+      <topic>camera_optical</topic>
       <gz_frame_id>camera_optical</gz_frame_id>
-      <camera>
-        <horizontal_fov>1.047</horizontal_fov>
-        <image>
-          <width>640</width>
-          <height>480</height>
-        </image>
-        <clip>
-          <near>0.1</near>
-          <far>100</far>
-        </clip>
-      </camera>
       <always_on>1</always_on>
       <update_rate>30</update_rate>
       <visualize>true</visualize>
-      <!-- <topic>camera</topic> -->
+      <camera>
+        <!-- Logitech C270 ≈ 55° horizontal FOV -->
+        <horizontal_fov>0.96</horizontal_fov>
+        <image>
+          <width>640</width> <!-- Logitech C270 ≈ 1280/2 -->
+          <height>360</height> <!-- Logitech C270 ≈ 720/2 -->
+          <format>R8G8B8</format>
+        </image>
+        <clip>
+          <near>0.2</near>
+          <far>20.0</far>
+        </clip>
+      </camera>
       <enable_metrics>true</enable_metrics>
     </sensor>
   </gazebo>
-  <gazebo>
-    <plugin
-      filename="gz-sim-diff-drive-system"
-      name="gz::sim::systems::DiffDrive">
-      <left_joint>left_wheel_joint</left_joint>
-      <right_joint>right_wheel_joint</right_joint>
-      <wheel_separation>0.236</wheel_separation>
-      <wheel_radius>0.034</wheel_radius>
-      <!--
-      Odometry in the diff drive plugin is quite bad, therefore
-      a dedicated OdometryPublisher plugin is being used.
-      As it can not be disabled we publish odom info to an unused topic
-      -->
-      <odom_topic>/unused/diff_drive_odometry</odom_topic>
-      <tf_topic>/unused/diff_drive_tf</tf_topic>
-      <odom_publish_frequency>1</odom_publish_frequency>
-      <frame_id>unused_odom_diff_drive</frame_id>
-      <child_frame_id>base_link</child_frame_id>
-    </plugin>
-  </gazebo>
-  <!-- OdometryPublisher being used instead of Diff Drive's odometry -->
-  <gazebo>
-    <plugin
-      filename="gz-sim-odometry-publisher-system"
-      name="gz::sim::systems::OdometryPublisher">
-      <odom_publish_frequency>60</odom_publish_frequency>
-      <robot_base_frame>base_link</robot_base_frame>
-      <odom_frame>odom</odom_frame>
-    </plugin>
-  </gazebo>
-  <gazebo>
-    <plugin
-      filename="gz-sim-joint-state-publisher-system"
-      name="gz::sim::systems::JointStatePublisher">
-      <joint_name>left_wheel_joint</joint_name>
-      <joint_name>right_wheel_joint</joint_name>
-    </plugin>
-  </gazebo>
 </robot>

File: mobo_bot_description/urdf/robot_urdf.xacro (robot description, xacro)
@@ -1,6 +1,6 @@
 <?xml version="1.0"?>
-<robot name="mobo_bot" xmlns:xacro="http://www.ros.org/wiki/xacro">
+<robot name="mobo_bot" xmlns:xacro="http://www.ros.org/wiki/xacro" xmlns:gz="http://gazebosim.org/schema">
     <xacro:arg name="run_gz_sim" default="false"/>
-    <xacro:arg name="base_type" default="2WHEEL"/>
+    <xacro:arg name="base_type" default="2WD"/>
     <xacro:property name="MOBOBOT_BASE_TYPE" value="$(arg base_type)"/>
     <material name="orange">
@@ -49,30 +49,40 @@
         </inertial>
     </xacro:macro>
+    <xacro:include filename="$(find mobo_bot_description)/urdf/robot_gazebo_properties.xacro" />
     <!-- Conditional inclusion -->
-    <xacro:if value="${MOBOBOT_BASE_TYPE == '2WHEEL'}">
-        <xacro:include filename="$(find mobo_bot_description)/urdf/2wheel_base/robot.xacro" />
+    <xacro:if value="${MOBOBOT_BASE_TYPE == '2WD'}">
+        <xacro:include filename="$(find mobo_bot_description)/urdf/2WD/robot.xacro" />
         <xacro:if value="$(arg run_gz_sim)">
-            <xacro:include filename="$(find mobo_bot_description)/urdf/2wheel_base/gazebo_properties.xacro" />
+            <xacro:include filename="$(find mobo_bot_description)/urdf/2WD/gazebo_control.xacro" />
         </xacro:if>
         <xacro:unless value="$(arg run_gz_sim)">
-            <xacro:include filename="$(find mobo_bot_description)/urdf/2wheel_base/ros2_control.xacro" />
+            <xacro:include filename="$(find mobo_bot_description)/urdf/2WD/ros2_control.xacro" />
         </xacro:unless>
     </xacro:if>
-    <xacro:if value="${MOBOBOT_BASE_TYPE == '2WHEEL_STD'}">
-        <xacro:include filename="$(find mobo_bot_description)/urdf/2wheel_std_base/robot.xacro" />
+    <xacro:if value="${MOBOBOT_BASE_TYPE == '4WD'}">
+        <xacro:include filename="$(find mobo_bot_description)/urdf/4WD/robot.xacro" />
         <xacro:if value="$(arg run_gz_sim)">
-            <xacro:include filename="$(find mobo_bot_description)/urdf/2wheel_std_base/gazebo_properties.xacro" />
+            <xacro:include filename="$(find mobo_bot_description)/urdf/4WD/gazebo_control.xacro" />
         </xacro:if>
         <xacro:unless value="$(arg run_gz_sim)">
-            <xacro:include filename="$(find mobo_bot_description)/urdf/2wheel_std_base/ros2_control.xacro" />
+            <xacro:include filename="$(find mobo_bot_description)/urdf/4WD/ros2_control.xacro" />
         </xacro:unless>
     </xacro:if>
-    <xacro:if value="${MOBOBOT_BASE_TYPE == '4WHEEL_STD'}">
-        <xacro:include filename="$(find mobo_bot_description)/urdf/4wheel_std_base/robot.xacro" />
+    <xacro:if value="${MOBOBOT_BASE_TYPE == 'MEC'}">
+        <xacro:include filename="$(find mobo_bot_description)/urdf/MEC/robot.xacro" />
         <xacro:if value="$(arg run_gz_sim)">
-            <xacro:include filename="$(find mobo_bot_description)/urdf/4wheel_std_base/gazebo_properties.xacro" />
+            <xacro:include filename="$(find mobo_bot_description)/urdf/MEC/gazebo_control.xacro" />
         </xacro:if>
         <xacro:unless value="$(arg run_gz_sim)">
-            <xacro:include filename="$(find mobo_bot_description)/urdf/4wheel_std_base/ros2_control.xacro" />
+            <xacro:include filename="$(find mobo_bot_description)/urdf/MEC/ros2_control.xacro" />
+        </xacro:unless>
+    </xacro:if>
+    <xacro:if value="${MOBOBOT_BASE_TYPE == '22WD'}">
+        <xacro:include filename="$(find mobo_bot_description)/urdf/22WD/robot.xacro" />
+        <xacro:if value="$(arg run_gz_sim)">
+            <xacro:include filename="$(find mobo_bot_description)/urdf/22WD/gazebo_control.xacro" />
+        </xacro:if>
+        <xacro:unless value="$(arg run_gz_sim)">
+            <xacro:include filename="$(find mobo_bot_description)/urdf/22WD/ros2_control.xacro" />
         </xacro:unless>
     </xacro:if>
