Commit message: update 2WD new wheel params

File: mobo_bot_description/urdf/2WD/robot.xacro (robot description, xacro)
@@ -13,7 +13,10 @@
     <xacro:property name="chassis_mass" value="2.0"/>
     <xacro:property name="chassis_color" value="orange"/>
-    <xacro:property name="wheel_seperation" value="0.207"/>
+    <!-- <xacro:property name="wheel_seperation" value="0.207"/>
     <xacro:property name="wheel_radius" value="0.033"/>
-    <xacro:property name="wheel_width" value="0.015"/>
+    <xacro:property name="wheel_width" value="0.015"/> -->
+    <xacro:property name="wheel_seperation" value="0.195"/>
+    <xacro:property name="wheel_radius" value="0.03"/>
+    <xacro:property name="wheel_width" value="0.008"/>
     <xacro:property name="wheel_mass" value="0.08"/>
     <xacro:property name="wheel_height_offset" value="0.01"/>
